Commit message: fixing devel

File: asv_launch/urdf/asv.xacro (robot description, xacro)
@@ -1,26 +1,82 @@
 <?xml version="1.0"?>
-<!-- STL-version of the URDF, used with gazebo for dynamic simulation  -->
 <robot name="asv" xmlns:xacro="http://www.ros.org/wiki/xacro">
     <xacro:property name="PI" value="3.1415926535897931"/>
-    <xacro:property name="eps" value="0.00000001"/>
+	<material name="blue">
+		<color rgba="0 0 0.8 0.5"/>
+	</material>
+	<material name="black">
+		<color rgba="0 0 0 0.8"/>
+	</material>
+	<material name="white">
+		<color rgba="1 1 1 1"/>
+	</material>
     <!-- Thruster link -->
-    <xacro:macro name="thruster_dummy_link" params="name xyz rpy">
-        <joint name="${name}" type="fixed">
+    <xacro:macro name="thruster_dummy_link" params="name xyz">
+        <joint name="${name}" type="revolute">
             <parent link="base_link"/>
             <child link="${name}"/>
-            <origin rpy="${rpy}" xyz="${xyz}"/>
+            <axis xyz="0 0 1"/>
+            <origin rpy="0 0 0" xyz="${xyz}"/>
+            <limit effort="20" lower="${-PI}" upper="${PI}" velocity="0"/>
         </joint>
         <link name="${name}">
-            <buoyancy><compensation>1.0</compensation></buoyancy>
-            <!--visual name="${name}">
+            <buoyancy><compensation>0.5</compensation></buoyancy>
+            <visual name="${name}">
                 <geometry>
-                    <cylinder length=".5" radius=".01"/>
+                    <cylinder length="0.1" radius=".1"/>
                 </geometry>
-                <material name="black">
-                    <color rgba="0 0 0 1"/>
-                </material>
+				<origin rpy="0 ${PI/2} 0" xyz="0 0 0"/>
+                <material name="black"/>
             </visual>
             <inertial>
                 <mass value=".1"/>
+                <inertia
+                    ixx=".1"
+                    ixy="0.0"
+                    ixz="0.0"
+                    iyy=".1"
+                    iyz="0.0"
+                    izz=".1"/>
+            </inertial>
+        </link>
+        <gazebo reference="${name}">
+            <material>Gazebo/Black</material>
+        </gazebo>
+    </xacro:macro>
+    <link name="base_link">
+    	<visual>
+            <geometry>
+                <box size="1.5 0.4 0.3"/>
+      		</geometry>
+            <material name="blue"/>
+        </visual>
+        <inertial>
+            <origin xyz="0 0 0" rpy="0 0 0"/>
+            <mass value="5"/>
+            <inertia
+                ixx="5"
+                ixy="0.0"
+                ixz="0.0"
+                iyy="5"
+                iyz="5"
+                izz="5"/>
+        </inertial>
+        <buoyancy>
+            <compensation>10.0</compensation>
+            <origin xyz = "0 0 0"/>
+            <limit radius="0.01"/>
+            <damping xyz="100 150 300" rpy="50 100 100"/>
+        </buoyancy>
+	</link>
+    <link name="thr0">
+        <buoyancy><compensation>0.0</compensation></buoyancy>
+        <visual name="thr0">
+            <geometry>
+                <cylinder length=".4" radius=".02"/>
+            </geometry>
+            <material name="white"/>
+        </visual>
+        <inertial>
+            <mass value=".5"/>
             <inertia
                 ixx=".1"
@@ -30,42 +86,13 @@
                 iyz="0.0"
                 izz=".1"/>
-            </inertial-->
-        </link>
-        <gazebo reference="${name}">
-            <material>Gazebo/Black</material>
-        </gazebo>
-    </xacro:macro>
-    <link name="base_link">
-        <visual>
-            <origin xyz="0 0 0" rpy="0 0 0"/>
-            <geometry>
-                <box size = "1.5 0.3 0.2"/>
-            </geometry>
-        </visual>
-        <inertial>
-            <origin xyz="0 0 0" rpy="0 0 0"/>
-            <mass value="15"/>
-            <inertia
-            ixx="15"
-            ixy="0.0"
-            ixz="0.0"
-            iyy="15"
-            iyz="5"
-            izz="15"/>
         </inertial>
-        <!--collision>
-        <origin xyz="0 0 0" rpy="0 0 0"/>
-        <geometry>
-        <box size="1 1 1"/>
-        </geometry>
-        </collision-->
-        <buoyancy>
-            <compensation>1.0</compensation>
-            <origin xyz= "0 0 0"/>
-            <limit radius="0.0"/>
-            <damping xyz="100 200 150" rpy="50 50 50"/>
-        </buoyancy>
     </link>
-    <xacro:thruster_dummy_link name="thr1" xyz="-0.5 0.115 -0.5" rpy="-0.0 -1.57079632679 0.0"/>
-    <xacro:thruster_dummy_link name="thr2" xyz="0.5 -0.115 -0.5" rpy="-0.0 -1.57079632679 0.0"/>
+    <joint name="thr0" type="revolute">
+        <parent link="base_link"/>
+        <child link="thr0"/>
+        <origin rpy="0 0 0" xyz="0.5 0 -0.05"/>
+        <limit effort="10" lower="${PI/2}" upper="${PI/2}" velocity="0"/>
+    </joint>
+    <xacro:thruster_dummy_link name="thr1" xyz="-0.7 -0.15 -0.2"/>
+    <xacro:thruster_dummy_link name="thr2" xyz="-0.7 0.15 -0.2"/>
 </robot>
